File: wsb-mega-shield.sch (KiCad schematic (older format))
At the start: 14 parts

Commit message: Finshed PCB, sent to china.
Parts:
- removed JP1: JUMPER-2SMD-NO, SparkFun-SJ_2S-NO, symbol JUMPER-2SMD-NO
- added C1: C, symbol C
- gave numbers to parts that had none: 4
Connections:
- net +12V: now also SHIELD1.V_IN
- net +3.3V: now also C1.2
- net GND: now also C1.1
